File: TEST PRAAN/STM32F103/STM32F103.kicad_sch (KiCad schematic)
At the start: 37 parts

Commit message: UPDATE
Parts:
- added R5, R6: 1K, Resistor_SMD:R_0805_2012Metric_Pad1.20x1.40mm_HandSolder, symbol Device:R_Small_US
- J3: renamed from J?; footprint (none) -> Connector_PinHeader_2.54mm:PinHeader_2x03_P2.54mm_Vertical
- RV1: renamed from RV?; footprint (none) -> Potentiometer_THT:Potentiometer_Bourns_3266W_Vertical
- SW1: renamed from SW?; footprint (none) -> Button_Switch_THT:SW_PUSH_6mm_H5mm
- gave numbers to parts that had none: 34
Connections:
- net +3V3: now also R5.1, R6.1
- net USB D+: now also U3.22 (PB11)
- net USB D-: now also U3.25 (PB12)
- net FAN: now reaches U3.10 (PA0)
- net TX: now reaches U3.12 (PA2)
- net RX: now reaches U3.13 (PA3)
- net TX1: now reaches U3.30 (PA9)
- net RX1: now reaches U3.31 (PA10)
- net SCL: now reaches U3.45 (PB8)
- net SCL: now also R5.2
- net SDA: now reaches U3.46 (PB9)
- net SDA: now also R6.2
- net +12V: now reaches D1.2 (A2), D2.1 (A), J1.1 (Pin_1)
- no-connect marks 1 -> 24
Other:
- note added: "I2C SENSOR"
- note added: "PMS7003 Sensor"
- note added: "SIMCOM7600"
